File: PulseCounter_Hardware/PulseCounter_Hardware.sch (KiCad schematic (older format))
At the start: 21 parts, among them U1 74LV8154, U10 74LV8154, U11 74LV8154, U12 MCP23008-E_P, U13 MCP23008-E_P, U14 74LV8154, U15 74LV8154, U16 MCP23008-E_P, U17 MCP23008-E_P, U2 74LV8154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

Commit message: Added I2C1 and I2C2 bus
Parts:
- removed U1, U10, U11, U14, U15, U2, U6, U7: 74LV8154, symbol 74xx:74LV8154
- removed U12, U13, U16, U17, U3, U4, U8, U9: MCP23008-E_P, digikey-footprints:DIP-18_W7.62mm, symbol dk_Interface-I-O-Expanders:MCP23008-E_P
Other:
- moved on the sheet: D1, R1, R2, RV1, U5
